Commit message: planar plugin successful.. ros2_control needs work

File: install/rcup_simulations/share/rcup_simulations/urdf/ArmPlate.urdf (robot description, URDF)
Before this commit: robot ArmPlate, 51 links, 50 joints
Links:
- added link imu_link, mass 0.1
Joints:
- added joint imu_joint: type fixed, parent base_footprint, child imu_link, origin xyz=0 0 0.01 rpy=0 0 0
